Commit message: obj+grasp cloud

File: grasp_point_model/Embodied lifting robot_two wheels_RM75-B-V/urdf/robot_hand.urdf (robot description, URDF)
Before this commit: robot Embodied lifting robot_two wheels_RM75-B-V, 16 links, 15 joints
Joints:
- joint joint_hand_base2: origin xyz=0 0 0.0228 rpy=0 0 0 -> xyz=0 0 0.0228 rpy=0 0 -1.57
